File: v2/pcb/pcb.kicad_sch (KiCad schematic)
At the start: 0 parts

Commit message: create v2 init, v2.json for VIA
Other:
- title: (none) -> maggie42cs
Changed lines of the file:
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@@
 	(generator_version "8.0")
 	(paper "A4")
+	(title_block
+		(title "maggie42cs")
+		(rev "2.0.1")
+	)
 	(sheet
 		(at 21.59 166.37)
