File: v2/pcb/left.kicad_sch (KiCad schematic)
At the start: 77 parts, among them J1 AudioJack3, J2 USB_C_Receptacle_USB2.0_16P, J3 Conn_01x03_Pin, SW1 SW_PUSH, SW10 SW_PUSH, SW11 SW_PUSH, SW12 SW_PUSH, SW13 SW_PUSH, SW14 SW_PUSH, SW15 SW_PUSH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

Commit message: create v2 init, v2.json for VIA
Parts:
- C10, C11, C12, C7, C8, C9: LCSC (none) -> C1525
- C13, C14: value 2.2F -> 2.2uF
- D10, D11, D12, D13, D14, D15, D16, D17, D18, D19, D2, D20, D21, D3, D4, D5, D6, D7, D8, D9: LCSC (none) -> C81598
- J1: footprint kbd:PJ-398A-5A_PJ-399B-6A -> kbd:MJ-4PP-9_1side; symbol Connector_Audio:AudioJack3 -> kbd:MJ-4PP-9; LCSC C128994 -> C22459514
- J2: footprint kbd:TYPE-C-31-M-13C -> Connector_USB:USB_C_Receptacle_HRO_TYPE-C-31-M-12; LCSC C2848620 -> C165948
Connections:
- net +5V: now also J1.D; no longer J1.T
- net CONN: now also J1.B; no longer J1.R
- net GND: now also J1.A; no longer J1.S
- net VBUS: now reaches F1.1, J2.A4 (VBUS), J2.A9 (VBUS), J2.B4 (VBUS), J2.B9 (VBUS)
- no-connect marks 21 -> 22
Other:
- title: (none) -> maggie42cs

Commit message: 1.1: create garbar files, 2.0: create left pcb
Other:
- moved on the sheet: C1, C12, C2, F1, R1, R4, R5, SD1, SMDSW1, STLED1, U1

Commit message: WIP: v2 refactoring
Parts:
- added C31, C32: C_Small, Capacitor_SMD:C_0603_1608Metric, symbol Device:C_Small
- added R17: 5.6k, Resistor_SMD:R_0603_1608Metric, symbol Device:R_Small
- added R18: 10k, Resistor_SMD:R_0402_1005Metric, symbol Device:R_Small
- SMDSW1, SMDSW2: footprint kbd:TS-1088R-02026 -> Button_Switch_SMD:SW_Push_1P1T_XKB_TS-1187A; LCSC C455280 -> C318884
- STLED1: footprint LED_SMD:LED_0402_1005Metric -> LED_SMD:LED_0603_1608Metric; LCSC C130723 -> C2290
- SW1: footprint kbd:CherryMX_ChocV2_Hotswap_1.5u -> kbd:keyswitch_cherrymx_choc12_hotswap_1.5u
- SW10, SW11, SW12, SW14, SW15, SW16, SW17, SW18, SW2, SW20, SW3, SW4, SW5, SW6, SW8, SW9: footprint kbd:CherryMX_ChocV2_Hotswap -> kbd:keyswitch_cherrymx_choc12_hotswap_1u
- SW13, SW19, SW21, SW7: footprint kbd:CherryMX_ChocV2_Hotswap_1.25u -> kbd:keyswitch_cherrymx_choc12_hotswap_1.25u
- U2: value W25Q128JVSIQ -> W25Q128JVS; footprint Package_SO:SOIC-8W_5.3x5.3mm_P1.27mm -> Package_SO:SOIC-8_5.23x5.23mm_P1.27mm; LCSC C97521 -> (none)
- Y1: footprint Crystal:Resonator_SMD_Murata_CSTxExxV-3Pin_3.0x1.1mm -> Crystal:Crystal_SMD_3225-4Pin_3.2x2.5mm; symbol Device:Crystal_GND2_Small -> Device:Crystal_GND24_Small; LCSC C341520 -> C9002
Connections:
- net CONN: now also J1.C; no longer J1.B
- net D+: now also J2.A6 (D+), J2.B6 (D+); no longer J2.A7 (D-), J2.B7 (D-)
- net D-: now also J2.A7 (D-), J2.B7 (D-); no longer J2.A6 (D+), J2.B6 (D+)
- net GND: now also Y1.4, C31.1, C32.1, R18.2
- net at R8.1, Y1.3: now also C32.2
- net at U3.20 (XIN), Y1.1: now also C31.2
- net SPLIT_USB_DETECT: now reaches U3.36 (GPIO24)
- net SPLIT_USB_DETECT: now also R17.2, R18.1
- net at F1.2, SD1.2 (A): now also R17.1
- no-connect marks 22 -> 21
Other:
- moved on the sheet: C1, C12, C15, C2, C3, D1, D10, D11, D12, D13, D14, D15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
