File: v2/pcb/right.kicad_sch (KiCad schematic)
At the start: 77 parts, among them J4 AudioJack3, J5 USB_C_Receptacle_USB2.0_16P, J6 Conn_01x03_Pin, SW22 SW_PUSH, SW23 SW_PUSH, SW24 SW_PUSH, SW25 SW_PUSH, SW26 SW_PUSH, SW27 SW_PUSH, SW28 SW_PUSH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

Commit message: create v2 init, v2.json for VIA
Parts:
- C23, C24, C25, C26, C27, C28: LCSC (none) -> C1525
- C29, C30: value 2.2F -> 2.2uF
- D23, D24, D25, D26, D27, D28, D29, D30, D31, D32, D33, D34, D35, D36, D37, D38, D39, D40, D41, D42: LCSC (none) -> C81598
- J4: footprint kbd:PJ-398A-5A_PJ-399B-6A -> kbd:MJ-4PP-9_1side; symbol Connector_Audio:AudioJack3 -> kbd:MJ-4PP-9; LCSC C128994 -> C22459514
- J5: footprint kbd:TYPE-C-31-M-13C -> Connector_USB:USB_C_Receptacle_HRO_TYPE-C-31-M-12; LCSC C2848620 -> C165948
Connections:
- net r+5V: now also J4.D; no longer J4.T
- net rCONN: now also J4.B; no longer J4.R
- net rGND: now also J4.A; no longer J4.S
- net VBUSR: now reaches F2.1, J5.A4 (VBUS), J5.A9 (VBUS), J5.B4 (VBUS), J5.B9 (VBUS)
- no-connect marks 21 -> 22
Other:
- title: (none) -> maggie42cs

Commit message: WIP: v2 refactoring
Parts:
- SMDSW3, SMDSW4: footprint kbd:TS-1088R-02026 -> Button_Switch_SMD:SW_Push_1P1T_XKB_TS-1187A
- SW22, SW23, SW24, SW25, SW26, SW28, SW29, SW30, SW31, SW32, SW33, SW34, SW35, SW36, SW37, SW38, SW41: footprint kbd:CherryMX_ChocV2_Hotswap -> kbd:keyswitch_cherrymx_choc12_hotswap_1u
- SW27: footprint kbd:CherryMX_ChocV2_Hotswap_1.5u -> kbd:keyswitch_cherrymx_choc12_hotswap_1.5u
- SW39, SW40, SW42: footprint kbd:CherryMX_ChocV2_Hotswap_1.25u -> kbd:keyswitch_cherrymx_choc12_hotswap_1.25u
- U5: value W25Q128JVSIQ -> W25Q128JVS; footprint Package_SO:SOIC-8W_5.3x5.3mm_P1.27mm -> Package_SO:SOIC-8_5.23x5.23mm_P1.27mm; LCSC C97521 -> (none)
- Y2: footprint Crystal:Resonator_SMD_Murata_CSTxExxV-3Pin_3.0x1.1mm -> Crystal:Crystal_SMD_3225-4Pin_3.2x2.5mm
Connections:
- net rCONN: now also J4.C; no longer J4.B
- net rD+: now also J5.A6 (D+), J5.B6 (D+); no longer J5.A7 (D-), J5.B7 (D-)
- net rD-: now also J5.A7 (D-), J5.B7 (D-); no longer J5.A6 (D+), J5.B6 (D+)
Changed lines of the file:
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@@
 	)
 	(no_connect
-		(at 200.66 34.29)
-	)
-	(no_connect
 		(at 105.41 144.78)
 	)
@@
 	)
 	(no_connect
+		(at 200.66 35.56)
+	)
+	(no_connect
 		(at 105.41 165.1)
 	)
@@
 	(wire
 		(pts
+			(xy 201.93 31.75) (xy 200.66 31.75)
+		)
+		(stroke
+			(width 0)
+			(type default)
+		)
+	)
+	(wire
+		(pts
 			(xy 132.08 72.39) (xy 140.97 72.39)
 		)
@@
 	(wire
 		(pts
+			(xy 203.2 27.94) (xy 203.2 33.02)
+		)
+		(stroke
+			(width 0)
+			(type default)
+		)
+	)
+	(wire
+		(pts
 			(xy 184.15 162.56) (xy 205.74 162.56)
 		)
@@
 	(wire
 		(pts
-			(xy 200.66 35.56) (xy 200.66 38.1)
-		)
-		(stroke
-			(width 0)
-			(type default)
-		)
-	)
-	(wire
-		(pts
 			(xy 227.33 124.46) (xy 248.92 124.46)
 		)
@@
 	(wire
 		(pts
-			(xy 200.66 38.1) (xy 204.47 38.1)
+			(xy 96.52 67.31) (xy 105.41 67.31)
 		)
 		(stroke
@@
 	(wire
 		(pts
-			(xy 96.52 67.31) (xy 105.41 67.31)
+			(xy 203.2 33.02) (xy 200.66 33.02)
 		)
 		(stroke
@@
 	(wire
 		(pts
-			(xy 200.66 33.02) (xy 204.47 33.02)
+			(xy 200.66 34.29) (xy 207.01 34.29)
 		)
 		(stroke
@@
 	(wire
 		(pts
+			(xy 201.93 41.91) (xy 201.93 31.75)
+		)
+		(stroke
+			(width 0)
+			(type default)
+		)
+	)
+	(wire
+		(pts
 			(xy 60.96 26.67) (xy 63.5 26.67)
 		)
@@
 	(global_label "rCONN"
 		(shape input)
-		(at 204.47 38.1 0)
+		(at 207.01 34.29 0)
 		(fields_autoplaced yes)
 		(effects
@@
 		)
 		(property "Intersheetrefs" "${INTERSHEET_REFS}"
-			(at 213.5029 38.1 0)
+			(at 216.0429 34.29 0)
 			(effects
 				(font
@@
 	(global_label "rD+"
 		(shape input)
-		(at 48.26 41.91 0)
+		(at 48.26 46.99 0)
 		(fields_autoplaced yes)
 		(effects
@@
 		)
 		(property "Intersheetrefs" "${INTERSHEET_REFS}"
-			(at 54.8738 41.91 0)
+			(at 54.8738 46.99 0)
 			(effects
 				(font
@@
 	(global_label "rD-"
 		(shape input)
-		(at 48.26 46.99 0)
+		(at 48.26 41.91 0)
 		(fields_autoplaced yes)
 		(effects
@@
 		)
 		(property "Intersheetrefs" "${INTERSHEET_REFS}"
-			(at 54.8738 46.99 0)
+			(at 54.8738 41.91 0)
 			(effects
 				(font
@@
 			)
 		)
-		(property "Footprint" "kbd:CherryMX_ChocV2_Hotswap_1.25u"
+		(property "Footprint" "kbd:keyswitch_cherrymx_choc12_hotswap_1.25u"
 			(at 157.48 152.4 0)
 			(effects
@@
 			)
 		)
-		(property "Footprint" "kbd:CherryMX_ChocV2_Hotswap"
+		(property "Footprint" "kbd:keyswitch_cherrymx_choc12_hotswap_1u"
 			(at 243.84 95.25 0)
 			(effects
@@
 			)
 		)
-		(property "Footprint" "kbd:CherryMX_ChocV2_Hotswap"
+		(property "Footprint" "kbd:keyswitch_cherrymx_choc12_hotswap_1u"
 			(at 157.48 133.35 0)
 			(effects
@@
 			)
 		)
-		(property "Footprint" "kbd:CherryMX_ChocV2_Hotswap"
+		(property "Footprint" "kbd:keyswitch_cherrymx_choc12_hotswap_1u"
 			(at 200.66 133.35 0)
 			(effects
@@
 			)
 		)
-		(property "Footprint" "kbd:CherryMX_ChocV2_Hotswap"
+		(property "Footprint" "kbd:keyswitch_cherrymx_choc12_hotswap_1u"
 			(at 243.84 133.35 0)
 			(effects
@@
 			)
 		)
-		(property "Footprint" "kbd:CherryMX_ChocV2_Hotswap"
+		(property "Footprint" "kbd:keyswitch_cherrymx_choc12_hotswap_1u"
 			(at 157.48 114.3 0)
 			(effects
@@
 			)
 		)
-		(property "Footprint" "Crystal:Resonator_SMD_Murata_CSTxExxV-3Pin_3.0x1.1mm"
+		(property "Footprint" "Crystal:Crystal_SMD_3225-4Pin_3.2x2.5mm"
 			(at 49.53 142.24 0)
 			(effects
@@
 			)
 		)
-		(property "Footprint" "kbd:CherryMX_ChocV2_Hotswap"
+		(property "Footprint" "kbd:keyswitch_cherrymx_choc12_hotswap_1u"
 			(at 243.84 114.3 0)
 			(effects
@@
 			)
 		)
-		(property "Footprint" "kbd:CherryMX_ChocV2_Hotswap"
+		(property "Footprint" "kbd:keyswitch_cherrymx_choc12_hotswap_1u"
 			(at 222.25 114.3 0)
 			(effects
@@
 			)
 		)
-		(property "Footprint" "kbd:CherryMX_ChocV2_Hotswap"
+		(property "Footprint" "kbd:keyswitch_cherrymx_choc12_hotswap_1u"
 			(at 179.07 133.35 0)
 			(effects
@@
 			)
 		)
-		(property "Footprint" "kbd:TS-1088R-02026"
+		(property "Footprint" "Button_Switch_SMD:SW_Push_1P1T_XKB_TS-1187A"
 			(at 125.73 33.02 0)
 			(effects
@@
 			)
 		)
-		(property "Footprint" "kbd:CherryMX_ChocV2_Hotswap"
+		(property "Footprint" "kbd:keyswitch_cherrymx_choc12_hotswap_1u"
 			(at 179.07 152.4 0)
 			(effects
@@
 			)
 		)
-		(property "Footprint" "kbd:CherryMX_ChocV2_Hotswap"
+		(property "Footprint" "kbd:keyswitch_cherrymx_choc12_hotswap_1u"
 			(at 200.66 95.25 0)
 			(effects
@@
 			)
 		)
-		(property "Footprint" "kbd:CherryMX_ChocV2_Hotswap"
+		(property "Footprint" "kbd:keyswitch_cherrymx_choc12_hotswap_1u"
 			(at 179.07 114.3 0)
 			(effects
@@
 			)
 		)
-		(property "Footprint" "kbd:CherryMX_ChocV2_Hotswap"
+		(property "Footprint" "kbd:keyswitch_cherrymx_choc12_hotswap_1u"
 			(at 179.07 95.25 0)
 			(effects
@@
 			)
 		)
-		(property "Footprint" "kbd:CherryMX_ChocV2_Hotswap_1.25u"
+		(property "Footprint" "kbd:keyswitch_cherrymx_choc12_hotswap_1.25u"
 			(at 265.43 133.35 0)
 			(effects
@@
 	(symbol
 		(lib_id "power:GND")
-		(at 200.66 31.75 90)
+		(at 201.93 41.91 0)
 		(unit 1)
 		(exclude_from_sim no)
@@
 		(fields_autoplaced yes)
 		(property "Reference" "#PWR034"
-			(at 207.01 31.75 0)
+			(at 201.93 48.26 0)
 			(effects
 				(font
@@
 		)
 		(property "Value" "rGND"
-			(at 204.47 31.7499 90)
+			(at 204.47 43.1799 0)
 			(effects
 				(font
 					(size 1.27 1.27)
 				)
-				(justify right)
+				(justify left)
 			)
 		)
 		(property "Footprint" ""
-			(at 200.66 31.75 0)
+			(at 201.93 41.91 0)
 			(effects
 				(font
@@
 		)
 		(property "Datasheet" ""
-			(at 200.66 31.75 0)
+			(at 201.93 41.91 0)
 			(effects
 				(font
@@
 		)
 		(property "Description" "Power symbol creates a global label with name \"GND\" , ground"
-			(at 200.66 31.75 0)
+			(at 201.93 41.91 0)
 			(effects
 				(font
@@
 			)
 		)
-		(property "Footprint" "kbd:CherryMX_ChocV2_Hotswap_1.25u"
+		(property "Footprint" "kbd:keyswitch_cherrymx_choc12_hotswap_1.25u"
 			(at 200.66 152.4 0)
 			(effects
@@
 			)
 		)
-		(property "Footprint" "kbd:CherryMX_ChocV2_Hotswap"
+		(property "Footprint" "kbd:keyswitch_cherrymx_choc12_hotswap_1u"
 			(at 222.25 133.35 0)
 			(effects
@@
 			)
 		)
-		(property "Footprint" "kbd:CherryMX_ChocV2_Hotswap"
+		(property "Footprint" "kbd:keyswitch_cherrymx_choc12_hotswap_1u"
 			(at 200.66 114.3 0)
 			(effects
@@
 			)
 		)
-		(property "Footprint" "kbd:TS-1088R-02026"
+		(property "Footprint" "Button_Switch_SMD:SW_Push_1P1T_XKB_TS-1187A"
 			(at 49.53 86.36 0)
 			(effects
@@
 			)
 		)
-		(property "Footprint" "kbd:CherryMX_ChocV2_Hotswap"
+		(property "Footprint" "kbd:keyswitch_cherrymx_choc12_hotswap_1u"
 			(at 265.43 114.3 0)
 			(effects
@@
 			)
 		)
-		(property "Footprint" "kbd:CherryMX_ChocV2_Hotswap_1.5u"
+		(property "Footprint" "kbd:keyswitch_cherrymx_choc12_hotswap_1.5u"
 			(at 265.43 95.25 0)
 			(effects
@@
 			)
 		)
-		(property "Footprint" "kbd:CherryMX_ChocV2_Hotswap"
+		(property "Footprint" "kbd:keyswitch_cherrymx_choc12_hotswap_1u"
 			(at 157.48 95.25 0)
 			(effects
@@
 			)
 		)
-		(property "Value" "W25Q128JVSIQ"
+		(property "Value" "W25Q128JVS"
 			(at 161.29 46.9899 0)
 			(effects
@@
 			)
 		)
-		(property "Footprint" "Package_SO:SOIC-8W_5.3x5.3mm_P1.27mm"
-			(at 152.4 45.72 0)
+		(property "Footprint" "Package_SO:SOIC-8_5.23x5.23mm_P1.27mm"
+			(at 152.4 22.86 0)
 			(effects
 				(font
@@
 			)
 		)
-		(property "Datasheet" "http://www.winbond.com/resource-files/w25q128jv_dtr%20revc%2003272018%20plus.pdf"
-			(at 152.4 45.72 0)
+		(property "Datasheet" "https://www.winbond.com/resource-files/w25q128jv_dtr%20revc%2003272018%20plus.pdf"
+			(at 152.4 20.32 0)
 			(effects
 				(font
@@
 		)
 		(property "Description" "128Mb Serial Flash Memory, Standard/Dual/Quad SPI, SOIC-8"
-			(at 152.4 45.72 0)
-			(effects
-				(font
-					(size 1.27 1.27)
-				)
-				(hide yes)
-			)
-		)
-		(property "LCSC" "C97521"
-			(at 152.4 45.72 0)
+			(at 152.4 17.78 0)
 			(effects
 				(font
@@
 			)
 		)
-		(property "Footprint" "kbd:CherryMX_ChocV2_Hotswap"
+		(property "Footprint" "kbd:keyswitch_cherrymx_choc12_hotswap_1u"
 			(at 222.25 95.25 0)
 			(effects
@@
 	(symbol
 		(lib_id "power:+5V")
-		(at 204.47 33.02 270)
+		(at 203.2 27.94 0)
 		(unit 1)
 		(exclude_from_sim no)
@@
 		(dnp no)
 		(property "Reference" "#PWR038"
-			(at 200.66 33.02 0)
+			(at 203.2 31.75 0)
 			(effects
 				(font
@@
 		)
 		(property "Value" "r+5V"
-			(at 207.772 33.782 0)
+			(at 203.962 24.638 0)
 			(effects
 				(font
@@
 		)
 		(property "Footprint" ""
-			(at 204.47 33.02 0)
+			(at 203.2 27.94 0)
 			(effects
 				(font
@@
 		)
 		(property "Datasheet" ""
-			(at 204.47 33.02 0)
+			(at 203.2 27.94 0)
 			(effects
 				(font
@@
 		)
 		(property "Description" "Power symbol creates a global label with name \"+5V\""
-			(at 204.47 33.02 0)
+			(at 203.2 27.94 0)
 			(effects
 				(font
