File: pcb/keyplate_l.kicad_pcb (KiCad board)
At the start: 2 copper layers, 128.6 x 95.2 mm, 28 parts, among them SW1 SW_PUSH, SW10 SW_PUSH, SW11 SW_PUSH, SW12 SW_PUSH, SW13 SW_PUSH, SW14 SW_PUSH, SW15 SW_PUSH, SW16 SW_PUSH, SW17 SW_PUSH, SW18 SW_PUSH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

Commit message: 1.1: create garbar files, 2.0: create left pcb
Parts:
- moved Ref** 4.76 mm to (57.1, 16.7)
