File: v2/pcb_l/pcb_l.kicad_sch (KiCad schematic)
At the start: 80 parts, among them J1 AudioJack3, J2 USB_C_Receptacle_USB2.0_16P, J3 Conn_01x03_Pin, SW1 SW_PUSH, SW10 SW_PUSH, SW11 SW_PUSH, SW12 SW_PUSH, SW13 SW_PUSH, SW14 SW_PUSH, SW15 SW_PUSH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

Commit message: update: 2.0.1_pcb_l
Parts:
- J3: footprint Connector_PinHeader_2.54mm:PinHeader_1x03_P2.54mm_Vertical -> Connector_PinHeader_1.27mm:PinHeader_1x03_P1.27mm_Vertical
Connections:
- net D+: now also J2.A6 (D+), J2.B6 (D+); no longer J2.A7 (D-), J2.B7 (D-)
- net D-: now also J2.A7 (D-), J2.B7 (D-); no longer J2.A6 (D+), J2.B6 (D+)
Changed lines of the file:
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@@
 	(global_label "D-"
 		(shape input)
-		(at 46.99 43.18 0)
+		(at 46.99 38.1 0)
 		(fields_autoplaced yes)
 		(effects
@@
 		)
 		(property "Intersheetrefs" "${INTERSHEET_REFS}"
-			(at 52.8176 43.18 0)
+			(at 52.8176 38.1 0)
 			(effects
 				(font
@@
 	(global_label "D+"
 		(shape input)
-		(at 46.99 38.1 0)
+		(at 46.99 43.18 0)
 		(fields_autoplaced yes)
 		(effects
@@
 		)
 		(property "Intersheetrefs" "${INTERSHEET_REFS}"
-			(at 52.8176 38.1 0)
+			(at 52.8176 43.18 0)
 			(effects
 				(font
@@
 			)
 		)
-		(property "Footprint" "Connector_PinHeader_2.54mm:PinHeader_1x03_P2.54mm_Vertical"
+		(property "Footprint" "Connector_PinHeader_1.27mm:PinHeader_1x03_P1.27mm_Vertical"
 			(at 24.13 172.72 0)
 			(effects
