File: v2/pcb_r/pcb_r.kicad_sch (KiCad schematic)
At the start: 80 parts, among them J1 AudioJack3, J2 USB_C_Receptacle_USB2.0_16P, J3 Conn_01x03_Pin, SW1 SW_PUSH, SW10 SW_PUSH, SW11 SW_PUSH, SW12 SW_PUSH, SW13 SW_PUSH, SW14 SW_PUSH, SW15 SW_PUSH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

Commit message: WIP: v2 refactoring
Parts:
- SW1: footprint kbd:CherryMX_ChocV2_Hotswap_1.5u -> kbd:keyswitch_cherrymx_choc12_hotswap_1u
- SW10, SW11, SW12, SW14, SW15, SW16, SW17, SW2, SW20, SW3, SW4, SW5, SW8, SW9: footprint kbd:CherryMX_ChocV2_Hotswap -> kbd:keyswitch_cherrymx_choc12_hotswap_1u
- SW13, SW7: footprint kbd:CherryMX_ChocV2_Hotswap_1.25u -> kbd:keyswitch_cherrymx_choc12_hotswap_1u
- SW18: footprint kbd:CherryMX_ChocV2_Hotswap -> kbd:keyswitch_cherrymx_choc12_hotswap_1.25u
- SW19, SW21: footprint kbd:CherryMX_ChocV2_Hotswap_1.25u -> kbd:keyswitch_cherrymx_choc12_hotswap_1.25u
- SW6: footprint kbd:CherryMX_ChocV2_Hotswap -> kbd:keyswitch_cherrymx_choc12_hotswap_1.5u
Connections:
- net COL0: now also SW19.1
- net COL1: now also SW20.1
- net COL2: now also SW21.1
- net COL3: no longer SW19.1
- net COL4: no longer SW20.1
- net COL5: no longer SW21.1
Other:
- moved on the sheet: D19, D20, D21, SW19, SW20, SW21
